File: cpu.sch (EAGLE design)
At the start: 24 parts, among them Q1 DMG2307LSOT23, U1 OPA2340EA/250, X1 ED060SC4_EINK, X2 PIIKKIRIMA-5

Commit message: Schematic should be complete
Schematic should have all parts now
Parts:
- removed D1: STM32L151VBT6, ST Microelctronics_By_element14_Batch_1:STM32L151VBT6
- added C10, C11, C12, C13, C8, C9: (no value), rcl:C-EUC0603
- added C14, C15, C18, C19, C20, C21, C7: (no value), rcl:C-EUC0805
- added C16, C17: 47n, rcl:C-EUC0805
- added E1, E2, E3: TB_ROUND, OMAT_IC:TB_ROUND
- added H1, H2, H3, H4, H5: (no value), OMAT_IC:LEDCHIP-LED0603
- added N4: MCP1700T-3302E/TT, Microchip_By_element14_Batch_1:MCP1700T-3302E/TT
- added N5: MAX412CPAMSOP, OMAT_IC:MAX412CPAMSOP
- added Q2: DMG2307LSOT23, OMAT_IC:DMG2307LSOT23
- added R10, R11, R12, R13, R14, R19, R20, R21, R22, R23, R24, R25, R26, R27, R28, R29, R30, R31, R8, R9: (no value), rcl:R-EU_R0603
- added R15, R32: 5k11, rcl:R-EU_R0603
- added R16, R17, R18: 22R, rcl:R-EU_R0603
- added U$1: ADP5063, OMAT_IC:ADP5063
- added U$2: DAFUG, dafug:DAFUG
- added X3, X7, X8, X9: PIIKKIRIMA-2, OMAT_IC:PIIKKIRIMA-2
- added X4: 629105136821, OMAT_IC:629105136821
- added X5: 693071010811, OMAT_IC:693071010811
- added X6: PIIKKIRIMA-6, OMAT_IC:PIIKKIRIMA-6
- U1: value OPA2340EA/250 -> STM32L151R8T6; device OMAT_IC:OPA2340EA/250 -> ST Microelctronics_By_element14_Batch_1:STM32L151R8T6
Connections:
- new net +3V3: C10.1, C11.1, C12.1, C13.1, C15.1, C8.1, C9.1, N4.VOUT, Q2.S, R10.2, R11.1, R12.1, R13.1, R14.1, R27.1, R28.1, R31.2, U1.VDDA, U1.VDD_1, U1.VDD_2, U1.VDD_3, U1.VDD_4, U1.VLCD, X3.1, X5.VDD
- new net +5V: R26.2
- new net BOOT0: R20.2, U1.BOOT0, X3.2
- new net CKV: U1.PB3, X1.U1CKV, X1.U2CKV
- new net CL: U1.PB4, X1.CL
- new net DACOUT1: R32.1, U1.PA4
- new net EINKD0: U1.PB8, X1.D0
- new net EINKD1: U1.PB9, X1.D1
- new net EINKD2: U1.PB10, X1.D2
- new net EINKD3: U1.PB11, X1.D3
- new net EINKD4: U1.PB12, X1.D4
- new net EINKD5: U1.PB13, X1.D5
- new net EINKD6: U1.PB14, X1.D6
- new net EINKD7: U1.PB15, X1.D7
- new net G8IO1: R21.1
- new net G8IO2: R22.1
- new net G8IO3: R23.1
- new net G8IO4: C16.1
- new net G9IO1: R24.2, U1.PC4
- new net G9IO2: C17.1, U1.PC5
- new net GMODE: U1.PB1, X1.GMODE1, X1.GMODE2
- new net LE: U1.PB5, X1.LE
- new net MISO1: U1.PA6, X5.DAT0/DO
- new net MOSI1: U1.PA7, X5.CMD/DI
- new net N$10: H1.A, R11.2
- new net N$12: H1.C, U1.PC8
- new net N$13: H2.A, R12.2
- new net N$14: H2.C, U1.PC9
- new net N$15: H3.A, R13.2
- new net N$16: H3.C, U1.PC10
- new net N$17: H4.A, R14.2
- new net N$18: N5B.-IN, R15.1, R32.2
- new net N$19: H4.C, U1.PC11
- new net N$20: H5.C, U$1.ILED
- new net N$21: C19.1, U$1.CBP
- new net N$22: H5.A, R25.1
- new net N$24: R26.1, U$1.DIGIO3
- new net N$4: R16.2, X4.2
- new net N$8: N5A.+IN, N5B.OUT, R15.2
- new net NSS1: U1.PA15, X5.CD/DAT3/CS
- new net OE: U1.PB6, X1.OE
- new net RESETN: R31.1, U1.NRST, X6.1
- new net RX1: U1.PA10, X6.6
- new net SCK1: R18.2, X5.CLK/SCLK
- new net SCL: R27.2, U$1.SCL
- new net SDA: R28.2, U$1.SDA
- new net SPH: U1.PB7, X1.SPH
- new net SPV/BOOT1: R19.2, U1.PB2, X1.U1SPV, X1.U2SPV
- new net STSCK1: R18.1, U1.PA5
- new net SWCLK: U1.PA14, X6.4
- new net SWDIO: U1.PA13, X6.2
- new net TB1: E1.1, R21.2
- new net TB2: E2.1, R22.2
- new net TB3: E3.1, R23.2
- new net TBSHIELD: R24.1
- new net TX1: U1.PA9, X6.5
- new net USBDM: R16.1, U1.PA11
- new net USBDP: R17.1, U1.PA12
- new net USD_DETN: U1.PA8, X5.DETECT
- new net VBATT: C21.1, R30.1, U$1.BATSNS, U$1.ISOB1, U$1.ISOB2, U$1.ISOB3, X7.1
- new net VEINK33: C7.1, Q2.D, X1.VDD
- new net VEINK33_CTRLN: Q2.G, R10.1, U1.PB0
- new net VEINKVCOM: N5A.-IN, N5A.OUT, X1.VCOM
- new net VSYS: C14.1, C20.1, N4.VIN, Q1.S, R1.2, R25.2, R29.2, R30.2, U$1.ISOS1, U$1.ISOS2, U$1.ISOS3
- new net VUSB: C18.1, R29.1, U$1.VIN1, U$1.VIN2, U$1.VIN3, X4.1, X9.1
- net GND: now also C10.2, C11.2, C12.2, C13.2, C14.2, C15.2, C16.2, C17.2, C18.2, C19.2, C20.2, C21.2, C7.2, C8.2, C9.2, N4.GND, N5B.+IN, R19.1, R20.1, R8.1, R9.1, U$1.AGND, X1.RL, X1.SHR, X1.U1CE1, X1.VBORDER, X4.5, X5.CASE, X5.VSS, X6.3, X7.2, X8.2, X9.2
- net N$2: now also R17.2, X4.3; no longer Q1.S, R1.2
- net VNEG15: now also N5A.V-, R9.2
- net VPOS15: now also N5A.V+, R8.2, X1.U1CE2, X1.U2CE1, X1.U2CE2
Other:
- note added: "3.3V REGULATOR"
- note added: "Charger Bypass Use only VBATT"
- note added: "DEBUG"
- note added: "EINK DISPLAY POWER SUPPLY"
- note added: "EINK VCOMMON DRIVER"
- note added: "KIMDLE V1.0 SEPT 2013 KL"
- note added: "LIPO CHARGER"
- note added: "LiPO Bypass Use only USB"
- note added: "MICRO SD CARD"
- note added: "No jumper = Boot normal Jumper = Bootloader USART"
- note added: "SPV is also BOOT1 and needs to be low when booting"
- note added: "STATUS/DIAG LEDS"
- note added: "Startup time > 3ms"
- note added: "TOUCH BUTTONS"
- note added: "USB"
- moved on the sheet: X1

Commit message: Buzzer added
Added smalles affordable buzzer.
Parts:
- added E4: AST7525MATRQ, OMAT_IC:AST7525MATRQ
- added R33, R34: (no value), rcl:R-EU_R0603
- added V2: DMG2307LSOT23, OMAT_IC:DMG2307LSOT23
Connections:
- removed net VEINK33_CTRLN: Q2.G, R10.1, U1.PB0
- new net BUZCTRLN: Q2.G, R10.1, R33.1, U1.PB0, U1.PC12, V2.G
- new net N$5: E4.-, R34.2
- new net VEINK1: E4.+, V2.D
- net +3V3: now also R33.2, V2.S
- net GND: now also R34.1
Changed lines of the file:
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@@
 <part name="GND37" library="supply1" deviceset="GND" device=""/>
 <part name="U$2" library="dafug" deviceset="DAFUG" device=""/>
+<part name="V2" library="OMAT_IC" deviceset="DMG2307L" device="SOT23"/>
+<part name="R33" library="rcl" deviceset="R-EU_" device="R0603"/>
+<part name="+3V11" library="supply1" deviceset="+3V3" device=""/>
+<part name="R34" library="rcl" deviceset="R-EU_" device="R0603"/>
+<part name="GND39" library="supply1" deviceset="GND" device=""/>
+<part name="E4" library="OMAT_IC" deviceset="AST7525MATRQ" device=""/>
 </parts>
 <sheets>
@@
 <instance part="GND37" gate="1" x="147.32" y="269.24"/>
 <instance part="U$2" gate="G$1" x="-116.84" y="350.52"/>
+<instance part="V2" gate="G$1" x="27.94" y="307.34"/>
+<instance part="R33" gate="G$1" x="15.24" y="317.5" rot="R90"/>
+<instance part="+3V11" gate="G$1" x="30.48" y="332.74"/>
+<instance part="R34" gate="G$1" x="30.48" y="279.4" rot="R90"/>
+<instance part="GND39" gate="1" x="30.48" y="271.78"/>
+<instance part="E4" gate="G$1" x="43.18" y="292.1"/>
 </instances>
 <busses>
@@
 <pinref part="X6" gate="G$1" pin="3"/>
 <pinref part="GND37" gate="1" pin="GND"/>
+</segment>
+<segment>
+<pinref part="R34" gate="G$1" pin="1"/>
+<pinref part="GND39" gate="1" pin="GND"/>
 </segment>
 </net>
@@
 </segment>
 </net>
-<net name="VEINK33_CTRLN" class="0">
+<net name="BUZCTRLN" class="0">
 <segment>
 <pinref part="Q2" gate="G$1" pin="G"/>
@@
 <label x="71.12" y="139.7" size="1.778" layer="95"/>
 <pinref part="U1" gate="A" pin="PB0"/>
+</segment>
+<segment>
+<pinref part="V2" gate="G$1" pin="G"/>
+<wire x1="25.4" y1="309.88" x2="15.24" y2="309.88" width="0.1524" layer="91"/>
+<pinref part="R33" gate="G$1" pin="1"/>
+<wire x1="15.24" y1="309.88" x2="-15.24" y2="309.88" width="0.1524" layer="91"/>
+<wire x1="15.24" y1="312.42" x2="15.24" y2="309.88" width="0.1524" layer="91"/>
+<junction x="15.24" y="309.88"/>
+<label x="-12.7" y="309.88" size="1.778" layer="95"/>
+</segment>
+<segment>
+<pinref part="U1" gate="A" pin="PC12"/>
+<wire x1="162.56" y1="167.64" x2="180.34" y2="167.64" width="0.1524" layer="91"/>
+<label x="165.1" y="167.64" size="1.778" layer="95"/>
 </segment>
 </net>
@@
 <wire x1="124.46" y1="292.1" x2="124.46" y2="294.64" width="0.1524" layer="91"/>
 <pinref part="+3V10" gate="G$1" pin="+3V3"/>
+</segment>
+<segment>
+<pinref part="R33" gate="G$1" pin="2"/>
+<wire x1="15.24" y1="322.58" x2="15.24" y2="325.12" width="0.1524" layer="91"/>
+<pinref part="V2" gate="G$1" pin="S"/>
+<wire x1="15.24" y1="325.12" x2="30.48" y2="325.12" width="0.1524" layer="91"/>
+<wire x1="30.48" y1="325.12" x2="30.48" y2="312.42" width="0.1524" layer="91"/>
+<pinref part="+3V11" gate="G$1" pin="+3V3"/>
+<wire x1="30.48" y1="330.2" x2="30.48" y2="325.12" width="0.1524" layer="91"/>
+<junction x="30.48" y="325.12"/>
 </segment>
 </net>
@@
 </segment>
 </net>
+<net name="VEINK1" class="0">
+<segment>
+<pinref part="V2" gate="G$1" pin="D"/>
+<wire x1="35.56" y1="294.64" x2="30.48" y2="294.64" width="0.1524" layer="91"/>
+<wire x1="30.48" y1="294.64" x2="30.48" y2="302.26" width="0.1524" layer="91"/>
+<pinref part="E4" gate="G$1" pin="+"/>
+</segment>
+</net>
+<net name="N$5" class="0">
+<segment>
+<wire x1="35.56" y1="292.1" x2="30.48" y2="292.1" width="0.1524" layer="91"/>
+<wire x1="30.48" y1="292.1" x2="30.48" y2="284.48" width="0.1524" layer="91"/>
+<pinref part="R34" gate="G$1" pin="2"/>
+<pinref part="E4" gate="G$1" pin="-"/>
+</segment>
+</net>

Commit message: Layout commit 1
First commit with some layout/placement
Parts:
- renumbered U$1 to N6
Connections:
- removed net +5V: R26.2
- net G8IO1: now also U1.PC0
- net G8IO2: now also U1.PC1
- net G8IO3: now also U1.PC2
- net G8IO4: now also U1.PC3
- net VSYS: now also R26.2, X8.1
Changed lines of the file:
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@@
 <part name="R23" library="rcl" deviceset="R-EU_" device="R0603"/>
 <part name="R24" library="rcl" deviceset="R-EU_" device="R0603"/>
-<part name="U$1" library="OMAT_IC" deviceset="ADP5063" device=""/>
+<part name="N6" library="OMAT_IC" deviceset="ADP5063" device=""/>
 <part name="C18" library="rcl" deviceset="C-EU" device="C0805"/>
 <part name="C19" library="rcl" deviceset="C-EU" device="C0805"/>
@@
 <part name="GND31" library="supply1" deviceset="GND" device=""/>
 <part name="R26" library="rcl" deviceset="R-EU_" device="R0603"/>
-<part name="P+3" library="supply1" deviceset="+5V" device=""/>
 <part name="C20" library="rcl" deviceset="C-EU" device="C0805"/>
 <part name="C21" library="rcl" deviceset="C-EU" device="C0805"/>
@@
 <instance part="R23" gate="G$1" x="327.66" y="96.52" rot="R90"/>
 <instance part="R24" gate="G$1" x="269.24" y="116.84" rot="R180"/>
-<instance part="U$1" gate="G$1" x="416.56" y="111.76"/>
+<instance part="N6" gate="G$1" x="416.56" y="111.76"/>
 <instance part="C18" gate="G$1" x="396.24" y="205.74"/>
 <instance part="C19" gate="G$1" x="396.24" y="182.88"/>
@@
 <instance part="GND31" gate="1" x="482.6" y="109.22"/>
 <instance part="R26" gate="G$1" x="403.86" y="142.24" rot="R180"/>
-<instance part="P+3" gate="1" x="386.08" y="147.32"/>
 <instance part="C20" gate="G$1" x="492.76" y="208.28"/>
 <instance part="C21" gate="G$1" x="492.76" y="182.88"/>
@@
 </segment>
 <segment>
-<pinref part="U$1" gate="G$1" pin="AGND"/>
+<pinref part="N6" gate="G$1" pin="AGND"/>
 <wire x1="474.98" y1="116.84" x2="482.6" y2="116.84" width="0.1524" layer="91"/>
 <wire x1="482.6" y1="116.84" x2="482.6" y2="111.76" width="0.1524" layer="91"/>
@@
 <segment>
 <wire x1="180.34" y1="198.12" x2="162.56" y2="198.12" width="0.1524" layer="91"/>
-<label x="165.1" y="198.12" size="1.778" layer="95"/>
+<label x="170.18" y="198.12" size="1.778" layer="95"/>
+<pinref part="U1" gate="A" pin="PC0"/>
 </segment>
 <segment>
@@
 <segment>
 <wire x1="180.34" y1="195.58" x2="162.56" y2="195.58" width="0.1524" layer="91"/>
-<label x="165.1" y="195.58" size="1.778" layer="95"/>
+<label x="170.18" y="195.58" size="1.778" layer="95"/>
+<pinref part="U1" gate="A" pin="PC1"/>
 </segment>
 <segment>
@@
 <segment>
 <wire x1="180.34" y1="193.04" x2="162.56" y2="193.04" width="0.1524" layer="91"/>
-<label x="165.1" y="193.04" size="1.778" layer="95"/>
+<label x="170.18" y="193.04" size="1.778" layer="95"/>
+<pinref part="U1" gate="A" pin="PC2"/>
 </segment>
 <segment>
@@
 <segment>
 <wire x1="180.34" y1="190.5" x2="162.56" y2="190.5" width="0.1524" layer="91"/>
-<label x="165.1" y="190.5" size="1.778" layer="95"/>
+<label x="170.18" y="190.5" size="1.778" layer="95"/>
+<pinref part="U1" gate="A" pin="PC3"/>
 </segment>
 <segment>
@@
 <pinref part="U1" gate="A" pin="PC4"/>
 <wire x1="162.56" y1="187.96" x2="180.34" y2="187.96" width="0.1524" layer="91"/>
-<label x="165.1" y="187.96" size="1.778" layer="95"/>
+<label x="170.18" y="187.96" size="1.778" layer="95"/>
 </segment>
 <segment>
@@
 <pinref part="U1" gate="A" pin="PC5"/>
 <wire x1="162.56" y1="185.42" x2="180.34" y2="185.42" width="0.1524" layer="91"/>
-<label x="165.1" y="185.42" size="1.778" layer="95"/>
+<label x="170.18" y="185.42" size="1.778" layer="95"/>
 </segment>
 <segment>
@@
 </segment>
 <segment>
-<pinref part="U$1" gate="G$1" pin="ISOS3"/>
+<pinref part="N6" gate="G$1" pin="ISOS3"/>
 <wire x1="474.98" y1="203.2" x2="480.06" y2="203.2" width="0.1524" layer="91"/>
 <wire x1="480.06" y1="203.2" x2="480.06" y2="208.28" width="0.1524" layer="91"/>
-<pinref part="U$1" gate="G$1" pin="ISOS1"/>
+<pinref part="N6" gate="G$1" pin="ISOS1"/>
 <wire x1="480.06" y1="208.28" x2="480.06" y2="213.36" width="0.1524" layer="91"/>
 <wire x1="480.06" y1="213.36" x2="474.98" y2="213.36" width="0.1524" layer="91"/>
 <wire x1="480.06" y1="213.36" x2="482.6" y2="213.36" width="0.1524" layer="91"/>
 <junction x="480.06" y="213.36"/>
-<pinref part="U$1" gate="G$1" pin="ISOS2"/>
+<pinref part="N6" gate="G$1" pin="ISOS2"/>
 <wire x1="482.6" y1="213.36" x2="492.76" y2="213.36" width="0.1524" layer="91"/>
 <wire x1="492.76" y1="213.36" x2="505.46" y2="213.36" width="0.1524" layer="91"/>
@@
 <label x="508" y="220.98" size="1.778" layer="95"/>
 <pinref part="C20" gate="G$1" pin="1"/>
-<wire x1="510.54" y1="215.9" x2="510.54" y2="220.98" width="0.1524" layer="91"/>
+<wire x1="510.54" y1="213.36" x2="510.54" y2="220.98" width="0.1524" layer="91"/>
 <wire x1="492.76" y1="213.36" x2="492.76" y2="210.82" width="0.1524" layer="91"/>
 <junction x="492.76" y="213.36"/>
@@
 <wire x1="505.46" y1="205.74" x2="505.46" y2="213.36" width="0.1524" layer="91"/>
 <junction x="505.46" y="213.36"/>
-<wire x1="546.1" y1="213.36" x2="510.54" y2="213.36" width="0.1524" layer="91"/>
-<wire x1="510.54" y1="213.36" x2="510.54" y2="215.9" width="0.1524" layer="91"/>
-</segment>
-</net>
-<net name="+5V" class="0">
+<wire x1="543.56" y1="213.36" x2="510.54" y2="213.36" width="0.1524" layer="91"/>
+<pinref part="X8" gate="G$1" pin="1"/>
+</segment>
 <segment>
 <pinref part="R26" gate="G$1" pin="2"/>
 <wire x1="398.78" y1="142.24" x2="386.08" y2="142.24" width="0.1524" layer="91"/>
 <wire x1="386.08" y1="142.24" x2="386.08" y2="144.78" width="0.1524" layer="91"/>
-<pinref part="P+3" gate="1" pin="+5V"/>
+<label x="383.54" y="144.78" size="1.778" layer="95"/>
 </segment>
 </net>
@@
 <net name="N$21" class="0">
 <segment>
-<pinref part="U$1" gate="G$1" pin="CBP"/>
+<pinref part="N6" gate="G$1" pin="CBP"/>
 <pinref part="C19" gate="G$1" pin="1"/>
 <wire x1="416.56" y1="187.96" x2="396.24" y2="187.96" width="0.1524" layer="91"/>
@@
 <net name="SCL" class="0">
 <segment>
-<pinref part="U$1" gate="G$1" pin="SCL"/>
+<pinref part="N6" gate="G$1" pin="SCL"/>
 <wire x1="416.56" y1="167.64" x2="375.92" y2="167.64" width="0.1524" layer="91"/>
 <label x="365.76" y="167.64" size="1.778" layer="95"/>
@@
 <net name="SDA" class="0">
 <segment>
-<pinref part="U$1" gate="G$1" pin="SDA"/>
+<pinref part="N6" gate="G$1" pin="SDA"/>
 <wire x1="416.56" y1="162.56" x2="383.54" y2="162.56" width="0.1524" layer="91"/>
 <label x="365.76" y="162.56" size="1.778" layer="95"/>
@@
 <segment>
 <pinref part="H5" gate="G$1" pin="C"/>
-<pinref part="U$1" gate="G$1" pin="ILED"/>
+<pinref part="N6" gate="G$1" pin="ILED"/>
 <wire x1="408.94" y1="116.84" x2="416.56" y2="116.84" width="0.1524" layer="91"/>
 </segment>
@@
 <net name="N$24" class="0">
 <segment>
-<pinref part="U$1" gate="G$1" pin="DIGIO3"/>
+<pinref part="N6" gate="G$1" pin="DIGIO3"/>
 <pinref part="R26" gate="G$1" pin="1"/>
 <wire x1="416.56" y1="142.24" x2="408.94" y2="142.24" width="0.1524" layer="91"/>
@@
 <net name="VBATT" class="0">
 <segment>
-<pinref part="U$1" gate="G$1" pin="ISOB3"/>
+<pinref part="N6" gate="G$1" pin="ISOB3"/>
 <wire x1="474.98" y1="177.8" x2="480.06" y2="177.8" width="0.1524" layer="91"/>
 <wire x1="480.06" y1="177.8" x2="480.06" y2="182.88" width="0.1524" layer="91"/>
-<pinref part="U$1" gate="G$1" pin="ISOB1"/>
+<pinref part="N6" gate="G$1" pin="ISOB1"/>
 <wire x1="480.06" y1="182.88" x2="480.06" y2="187.96" width="0.1524" layer="91"/>
 <wire x1="480.06" y1="187.96" x2="474.98" y2="187.96" width="0.1524" layer="91"/>
-<pinref part="U$1" gate="G$1" pin="ISOB2"/>
+<pinref part="N6" gate="G$1" pin="ISOB2"/>
 <wire x1="474.98" y1="182.88" x2="480.06" y2="182.88" width="0.1524" layer="91"/>
 <junction x="480.06" y="182.88"/>
 <wire x1="480.06" y1="187.96" x2="492.76" y2="187.96" width="0.1524" layer="91"/>
 <junction x="480.06" y="187.96"/>
-<pinref part="U$1" gate="G$1" pin="BATSNS"/>
+<pinref part="N6" gate="G$1" pin="BATSNS"/>
 <wire x1="492.76" y1="187.96" x2="505.46" y2="187.96" width="0.1524" layer="91"/>
 <wire x1="505.46" y1="187.96" x2="515.62" y2="187.96" width="0.1524" layer="91"/>
@@
 <net name="VUSB" class="0">
 <segment>
-<pinref part="U$1" gate="G$1" pin="VIN3"/>
+<pinref part="N6" gate="G$1" pin="VIN3"/>
 <wire x1="416.56" y1="203.2" x2="411.48" y2="203.2" width="0.1524" layer="91"/>
 <wire x1="411.48" y1="203.2" x2="411.48" y2="208.28" width="0.1524" layer="91"/>
-<pinref part="U$1" gate="G$1" pin="VIN1"/>
+<pinref part="N6" gate="G$1" pin="VIN1"/>
 <wire x1="411.48" y1="208.28" x2="411.48" y2="213.36" width="0.1524" layer="91"/>
 <wire x1="411.48" y1="213.36" x2="416.56" y2="213.36" width="0.1524" layer="91"/>
@@
 <junction x="411.48" y="213.36"/>
 <wire x1="408.94" y1="213.36" x2="396.24" y2="213.36" width="0.1524" layer="91"/>
-<pinref part="U$1" gate="G$1" pin="VIN2"/>
+<pinref part="N6" gate="G$1" pin="VIN2"/>
 <wire x1="416.56" y1="208.28" x2="411.48" y2="208.28" width="0.1524" layer="91"/>
 <junction x="411.48" y="208.28"/>

Commit message: All parts first time onboard - placed
Touchbuttons also prelocated for OSHpark testing
Parts:
- removed R29, R30: (no value), rcl:R-EU_R0603
- added SJ1, SJ2: (no value), OMAT_IC:SJ
- renumbered Q1 to V4, Q2 to V3, V2 to V5
Connections:
- new net EINKVDDCTRLN: R10.1, U1.PB0, V3.G
- net BUZCTRLN: no longer R10.1, U1.PB0, V3.G
- net VBATT: now also SJ2.1; no longer R30.1
- net VEINK33: now also X1.U1CE2, X1.U2CE1, X1.U2CE2
- net VPOS15: no longer X1.U1CE2, X1.U2CE1, X1.U2CE2
- net VSYS: now also SJ1.2, SJ2.2; no longer R29.2, R30.2
- net VUSB: now also SJ1.1; no longer R29.1

Commit message: Layout cont2
17 airwires left.
touch buttons removed from cpu board
Parts:
- removed E1, E2, E3: TB_ROUND, OMAT_IC:TB_ROUND
- removed R18: 22R, rcl:R-EU_R0603
- added C22: (no value), rcl:C-EUC0603
- added D2: TMP75DGK, ti_tmp:TMP75DGK
- added X10: PIIKKIRIMA-4, OMAT_IC:PIIKKIRIMA-4
- C19: device rcl:C-EUC0805 -> rcl:C-EUC0603
- renumbered U1 to D1
Connections:
- net N$12 renamed LED1
- net N$14 renamed LED2
- net N$16 renamed LED3
- net N$19 renamed LED4
- removed net STSCK1: D1.PA5, R18.1
- net +3V3: now also C22.1, D2.V+
- net GND: now also C22.2, D2.A0, D2.A1, D2.A2, D2.GND
- net OE: now also D1.PA1; no longer D1.PB6
- net SCK1: now also D1.PA5; no longer R18.2
- net SCL: now also D1.PB6, D2.SCL
- net SDA: now also D1.PB7, D2.SDA
- net SPH: now also D1.PA2; no longer D1.PB7
- net TB1: now also X10.2; no longer E1.1
- net TB2: now also X10.3; no longer E2.1
- net TB3: now also X10.4; no longer E3.1
- net TBSHIELD: now also X10.1
Other:
- note added: "TEMP SENSOR"
- note added: "TOUCH IF"
- note removed: "TOUCH BUTTONS"
- moved on the sheet: C16, C17, R21, R22, R23, R24

Commit message: Layout complete
First completed layout , Airwires 0
Connections:
- net +3V3: now also R25.2
- net VSYS: no longer R25.2
Changed lines of the file:
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@@
 <part name="C22" library="rcl" deviceset="C-EU" device="C0603"/>
 <part name="GND40" library="supply1" deviceset="GND" device=""/>
+<part name="+3V13" library="supply1" deviceset="+3V3" device=""/>
 </parts>
 <sheets>
@@
 <instance part="C22" gate="G$1" x="325.12" y="165.1"/>
 <instance part="GND40" gate="1" x="325.12" y="152.4"/>
+<instance part="+3V13" gate="G$1" x="378.46" y="121.92"/>
 </instances>
 <busses>
@@
 <junction x="325.12" y="170.18"/>
 </segment>
+<segment>
+<pinref part="R25" gate="G$1" pin="2"/>
+<wire x1="386.08" y1="116.84" x2="378.46" y2="116.84" width="0.1524" layer="91"/>
+<wire x1="378.46" y1="116.84" x2="378.46" y2="119.38" width="0.1524" layer="91"/>
+<pinref part="+3V13" gate="G$1" pin="+3V3"/>
+</segment>
 </net>
 <net name="EINKD0" class="0">
@@
 </segment>
 <segment>
-<pinref part="R25" gate="G$1" pin="2"/>
-<wire x1="386.08" y1="116.84" x2="365.76" y2="116.84" width="0.1524" layer="91"/>
-<label x="365.76" y="116.84" size="1.778" layer="95"/>
-</segment>
-<segment>
