File: cpu.sch (EAGLE design)
At the start: 89 parts, among them X1 ED060SC4_EINK, X10 PIIKKIRIMA-4, X2 PIIKKIRIMA-5, X3 PIIKKIRIMA-2, X4 629105136821, X5 693071010811, X6 PIIKKIRIMA-6, X7 PIIKKIRIMA-2, X8 PIIKKIRIMA-2, X9 PIIKKIRIMA-2

Commit message: Bypass, tuning
One 0805 bulk bypass added.
GND fills fixed close G1
Parts:
- added C25: (no value), rcl:C-EUC0805
Connections:
- net +3V3: now also C25.1
- net GND: now also C25.2
Changed lines of the file:
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@@
 <part name="C24" library="rcl" deviceset="C-EU" device="C0603"/>
 <part name="GND41" library="supply1" deviceset="GND" device=""/>
+<part name="C25" library="rcl" deviceset="C-EU" device="C0805"/>
+<part name="GND42" library="supply1" deviceset="GND" device=""/>
+<part name="+3V14" library="supply1" deviceset="+3V3" device=""/>
 </parts>
 <sheets>
@@
 <instance part="C24" gate="G$1" x="182.88" y="226.06"/>
 <instance part="GND41" gate="1" x="195.58" y="223.52"/>
+<instance part="C25" gate="G$1" x="-53.34" y="144.78"/>
+<instance part="GND42" gate="1" x="-53.34" y="137.16"/>
+<instance part="+3V14" gate="G$1" x="-53.34" y="149.86"/>
 </instances>
 <busses>
@@
 <wire x1="182.88" y1="228.6" x2="182.88" y2="231.14" width="0.1524" layer="91"/>
 <junction x="182.88" y="231.14"/>
+</segment>
+<segment>
+<pinref part="C25" gate="G$1" pin="2"/>
+<pinref part="GND42" gate="1" pin="GND"/>
 </segment>
 </net>
@@
 <pinref part="+3V13" gate="G$1" pin="+3V3"/>
 </segment>
-</net>
+<segment>
+<pinref part="C25" gate="G$1" pin="1"/>
+<pinref part="+3V14" gate="G$1" pin="+3V3"/>
+</segment>
+</net>

Commit message: Power control signals added
DCDC Converter enables (all three) were missing from schematic.
Processor grounds connected too.
Connections:
- net GND: now also D1.VSSA, D1.VSS_1, D1.VSS_2, D1.VSS_3, D1.VSS_4
- net VEINK_CTRLN: now also D1.PD2
- net VNEG_CTRLN: now also D1.PC7
- net VPOS_CTRLN: now also D1.PC6
Other:
- moved on the sheet: H1, H2, H3, H4, R11, R12, R13, R14

Commit message: Final - ready to order
Part values added
Parts:
- removed U$2: DAFUG, dafug:DAFUG
- C1, C14, C7: value (none) -> 1u 50V
- C10, C11, C12, C13, C19, C22, C8, C9: value (none) -> 100n
- C15, C18, C20, C21, C25: value (none) -> 10u 10V
- C2, C3, C4, C5, C6: value (none) -> 4u7 50V
- C23, C24: value (none) -> 12p
- H1, H2, H3: value (none) -> GRN
- H4, H5: value (none) -> YEL
- N5: value MAX412CPAMSOP -> LM358
- R1, R10, R19, R2, R20, R21, R22, R23, R24, R26, R31, R33, R4, R5, R6, R8, R9: value (none) -> 10k
- R11, R12, R13, R14, R25: value (none) -> 511R
- R15, R32: value 5k11 -> 10k
- R27, R28: value (none) -> 2k15
- R3: value (none) -> 165k
- R34: value (none) -> 22R
- R7: value (none) -> 160k
- V3, V4, V5: value DMG2307LSOT23 -> FDV304
Other:
- moved on the sheet: C3, C4, SJ2
