File: cpu.brd (EAGLE design)
At the start: 72.4 x 38.1 mm, 91 parts, among them X1 ED060SC4_EINK, X10 PIIKKIRIMA-4, X2 PIIKKIRIMA-5, X3 PIIKKIRIMA-2, X4 629105136821, X5 693071010811, X6 PIIKKIRIMA-6, X7 PIIKKIRIMA-2, X8 PIIKKIRIMA-2, X9 PIIKKIRIMA-2

Commit message: KIMDLE logo revisited
The imported bitmap was rejected by OSHpark. made my own from polygons
Parts:
- removed U$1: (no value), dafug:KIMDLE
Changed lines of the file:
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@@
 <layer number="22" name="bPlace" color="7" fill="1" visible="yes" active="yes"/>
 <layer number="23" name="tOrigins" color="15" fill="1" visible="no" active="yes"/>
-<layer number="24" name="bOrigins" color="15" fill="1" visible="no" active="yes"/>
+<layer number="24" name="bOrigins" color="15" fill="1" visible="yes" active="yes"/>
 <layer number="25" name="tNames" color="7" fill="1" visible="no" active="yes"/>
-<layer number="26" name="bNames" color="7" fill="1" visible="no" active="yes"/>
+<layer number="26" name="bNames" color="7" fill="1" visible="yes" active="yes"/>
 <layer number="27" name="tValues" color="7" fill="1" visible="no" active="yes"/>
 <layer number="28" name="bValues" color="7" fill="1" visible="no" active="yes"/>
@@
 <layer number="151" name="HeatSink" color="7" fill="1" visible="no" active="yes"/>
 <layer number="199" name="Contour" color="7" fill="1" visible="no" active="yes"/>
-<layer number="200" name="200bmp" color="1" fill="10" visible="yes" active="yes"/>
+<layer number="200" name="200bmp" color="1" fill="10" visible="no" active="yes"/>
 <layer number="201" name="201bmp" color="2" fill="10" visible="no" active="yes"/>
 <layer number="202" name="202bmp" color="3" fill="10" visible="no" active="yes"/>
@@
 <text x="5.08" y="33.3375" size="1.778" layer="21">+</text>
 <text x="19.431" y="33.3375" size="1.778" layer="21">+</text>
+<polygon width="0.1524" layer="22">
+<vertex x="51.1912375" y="17.148428125"/>
+<vertex x="47.888575" y="27.14109375"/>
+<vertex x="46.11021875" y="27.14109375"/>
+<vertex x="47.549840625" y="22.991596875"/>
+<vertex x="46.745346875" y="23.245646875"/>
+<vertex x="46.1525625" y="23.58438125"/>
+<vertex x="45.43275" y="24.17716875"/>
+<vertex x="44.797625" y="24.93931875"/>
+<vertex x="44.289521875" y="25.743815625"/>
+<vertex x="43.908446875" y="26.463625"/>
+<vertex x="43.612053125" y="27.098753125"/>
+<vertex x="43.40034375" y="27.5645125"/>
+<vertex x="40.478759375" y="27.26811875"/>
+<vertex x="42.08775" y="25.53210625"/>
+<vertex x="42.89224375" y="24.7276125"/>
+<vertex x="43.485028125" y="24.219509375"/>
+<vertex x="44.331865625" y="23.542040625"/>
+<vertex x="44.712940625" y="23.287990625"/>
+<vertex x="45.60211875" y="22.69520625"/>
+<vertex x="45.305725" y="21.890709375"/>
+<vertex x="45.094015625" y="21.128559375"/>
+<vertex x="44.92465" y="20.451090625"/>
+<vertex x="44.75528125" y="19.6889375"/>
+<vertex x="44.6706" y="19.096153125"/>
+<vertex x="44.62825625" y="18.249315625"/>
+<vertex x="44.6706" y="17.4871625"/>
+<vertex x="44.75528125" y="16.9790625"/>
+<vertex x="47.719209375" y="17.2331125"/>
+<vertex x="47.33813125" y="18.545709375"/>
+<vertex x="47.041740625" y="19.6889375"/>
+<vertex x="46.999396875" y="20.154696875"/>
+<vertex x="47.08408125" y="20.62045625"/>
+<vertex x="47.25345" y="20.959190625"/>
+<vertex x="47.46515625" y="21.128559375"/>
+<vertex x="47.973259375" y="21.297925"/>
+<vertex x="49.074146875" y="17.148428125"/>
+</polygon>
+<polygon width="0.1524" layer="22">
+<vertex x="43.14629375" y="17.275453125"/>
+<vertex x="41.325596875" y="17.275453125"/>
+<vertex x="41.029203125" y="18.799759375"/>
+<vertex x="40.69046875" y="20.23938125"/>
+<vertex x="40.394078125" y="21.382609375"/>
+<vertex x="39.5049" y="23.923115625"/>
+<vertex x="38.6580625" y="25.955521875"/>
+<vertex x="38.0229375" y="27.606853125"/>
+<vertex x="39.970659375" y="27.479828125"/>
+<vertex x="40.351734375" y="25.828496875"/>
+<vertex x="40.648128125" y="24.642928125"/>
+<vertex x="40.9868625" y="23.372675"/>
+<vertex x="41.621990625" y="21.382609375"/>
+</polygon>
+<polygon width="0.1524" layer="22">
+<vertex x="40.224709375" y="17.2331125"/>
+<vertex x="36.583315625" y="27.3104625"/>
+<vertex x="33.577046875" y="27.098753125"/>
+<vertex x="33.873440625" y="23.033940625"/>
+<vertex x="33.3653375" y="23.33033125"/>
+<vertex x="33.1112875" y="23.542040625"/>
+<vertex x="32.6031875" y="24.092484375"/>
+<vertex x="31.968059375" y="24.93931875"/>
+<vertex x="31.45995625" y="25.65913125"/>
+<vertex x="31.036540625" y="26.3366"/>
+<vertex x="30.82483125" y="26.802359375"/>
+<vertex x="30.613121875" y="27.26811875"/>
+<vertex x="28.36900625" y="27.26811875"/>
+<vertex x="30.0203375" y="22.991596875"/>
+<vertex x="30.2743875" y="22.187103125"/>
+<vertex x="30.443753125" y="21.59431875"/>
+<vertex x="30.740146875" y="20.451090625"/>
+<vertex x="30.994196875" y="19.604253125"/>
+<vertex x="31.20590625" y="18.8421"/>
+<vertex x="31.629325" y="17.3601375"/>
+<vertex x="33.53470625" y="17.3601375"/>
+<vertex x="32.941921875" y="18.503365625"/>
+<vertex x="32.518503125" y="19.4348875"/>
+<vertex x="32.095084375" y="20.49343125"/>
+<vertex x="31.798690625" y="21.46729375"/>
+<vertex x="31.544640625" y="22.314128125"/>
+<vertex x="31.33293125" y="23.033940625"/>
+<vertex x="30.95185625" y="24.55824375"/>
+<vertex x="34.508565625" y="19.39254375"/>
+<vertex x="36.11755625" y="19.4348875"/>
+<vertex x="35.8211625" y="25.4897625"/>
+<vertex x="36.49863125" y="23.4997"/>
+<vertex x="37.091415625" y="21.1709"/>
+<vertex x="37.47249375" y="19.900646875"/>
+<vertex x="37.938253125" y="18.58805"/>
+<vertex x="38.488696875" y="17.190771875"/>
+</polygon>
+<polygon width="0.1524" layer="22">
+<vertex x="24.55824375" y="16.04754375"/>
+<vertex x="22.82223125" y="20.705140625"/>
+<vertex x="22.314128125" y="22.314128125"/>
+<vertex x="20.705140625" y="27.5645125"/>
+<vertex x="18.03760625" y="27.5645125"/>
+<vertex x="19.477228125" y="24.81229375"/>
+<vertex x="20.578115625" y="22.610521875"/>
+<vertex x="21.72134375" y="20.11235625"/>
+<vertex x="22.6528625" y="17.741215625"/>
+<vertex x="22.82223125" y="17.275453125"/>
+<vertex x="18.03760625" y="18.16463125"/>
+<vertex x="18.334" y="15.793490625"/>
+</polygon>
+<polygon width="0.1524" layer="22">
+<vertex x="12.10975625" y="17.2331125"/>
+<vertex x="16.9790625" y="17.190771875"/>
+<vertex x="13.507034375" y="27.39514375"/>
+<vertex x="7.536840625" y="27.733878125"/>
+<vertex x="7.960259375" y="26.378940625"/>
+<vertex x="8.595384375" y="26.16723125"/>
+<vertex x="9.188171875" y="26.04020625"/>
+<vertex x="9.865640625" y="25.91318125"/>
+<vertex x="10.712475" y="25.828496875"/>
+<vertex x="11.771021875" y="25.743815625"/>
+<vertex x="12.575515625" y="25.701471875"/>
+<vertex x="13.1683" y="23.372675"/>
+<vertex x="11.051209375" y="23.372675"/>
+<vertex x="11.64399375" y="21.42495"/>
+<vertex x="14.1421625" y="21.42495"/>
+<vertex x="15.0313375" y="18.461025"/>
+<vertex x="13.84576875" y="18.461025"/>
+<vertex x="11.771021875" y="18.58805"/>
+</polygon>
+<polygon width="0.1524" layer="22">
+<vertex x="30.486096875" y="17.19076875"/>
+<vertex x="29.512234375" y="20.112353125"/>
+<vertex x="28.157296875" y="19.8159625"/>
+<vertex x="28.580715625" y="18.461025"/>
+<vertex x="27.903246875" y="18.58805"/>
+<vertex x="27.01406875" y="19.01146875"/>
+<vertex x="26.209575" y="19.6889375"/>
+<vertex x="25.701471875" y="20.36640625"/>
+<vertex x="25.15103125" y="21.467290625"/>
+<vertex x="24.8546375" y="22.22944375"/>
+<vertex x="24.68526875" y="23.0339375"/>
+<vertex x="24.6005875" y="23.83843125"/>
+<vertex x="24.642928125" y="24.473559375"/>
+<vertex x="24.7276125" y="24.896978125"/>
+<vertex x="24.8546375" y="25.1086875"/>
+<vertex x="25.066346875" y="25.278053125"/>
+<vertex x="25.320396875" y="25.3627375"/>
+<vertex x="26.04020625" y="25.405078125"/>
+<vertex x="26.675334375" y="25.3627375"/>
+<vertex x="28.11495625" y="19.9429875"/>
+<vertex x="29.46989375" y="20.23938125"/>
+<vertex x="27.01406875" y="27.26811875"/>
+<vertex x="26.378940625" y="27.26811875"/>
+<vertex x="25.65913125" y="27.225778125"/>
+<vertex x="25.066346875" y="27.056409375"/>
+<vertex x="24.346534375" y="26.717675"/>
+<vertex x="23.626725" y="26.16723125"/>
+<vertex x="23.20330625" y="25.4897625"/>
+<vertex x="22.991596875" y="24.93931875"/>
+<vertex x="22.94925625" y="23.923115625"/>
+<vertex x="23.118625" y="23.118621875"/>
+<vertex x="23.457359375" y="22.060078125"/>
+<vertex x="23.92311875" y="20.959190625"/>
+<vertex x="24.388878125" y="20.112353125"/>
+<vertex x="25.1086875" y="19.053809375"/>
+<vertex x="25.65913125" y="18.461025"/>
+<vertex x="26.548309375" y="17.78355625"/>
+<vertex x="27.225778125" y="17.444821875"/>
+<vertex x="28.030271875" y="17.2331125"/>
+<vertex x="29.004134375" y="17.1060875"/>
+<vertex x="29.85096875" y="17.1060875"/>
+</polygon>
 </plain>
 <attributes>
@@
 </element>
 <element name="U$3" library="dafug" package="DAFUG" value="" x="9.0805" y="9.906" rot="MR0"/>
-<element name="U$1" library="dafug" package="KIMDLE" value="" x="51.064209375" y="16.513303125" rot="MR0"/>
 </elements>
 <signals>
